File: schematic/hour-meter-board-compact/hour-meter-board-compact.kicad_pcb (KiCad board)
At the start: 2 copper layers, 80 x 70 mm, 115 parts, among them J101 VIN 9-36V, J102 PSU header, J201 USB-C, J301 VEHICLE IN, J501 WP, J701 RS485, J702 TERM, J703 BIAS, J801 UART, J802 GPS, J803 QWIIC, J804 EXP, Q201 MMBT3904, Q202 MMBT3904, SW201 RESET, SW202 BOOT, U201 ESP32-WROOM-32E-N4, U202 CH340C, U203 USBLC6-2SC6, U204 AMS1117-3.3, U301 PC817C-S, U302 PC817C-S, U401 DS3231MZ+TRL, U501 AT24C256 DIP-8 (socketed), U601 MPU-6500, U602 LIS3MDLTR, U701 THVD2410DR, U801 74LVC1G17GW, U802 SRV05-4

Commit message: feat(pcb): mark where JLCPCB prints the order number
- New add_order_mark() in the shared board builder: places the
  JLCJLCJLCJLC placeholder (1.0 mm, 0.15 mm stroke) at the free spot
  nearest a given point, clear of pads, holes, courtyards, silkscreen and
  the outline
- Compact board and PSU-B carry it on the bottom silkscreen; their build
  scripts put it back on a rebuild
- Regenerate both boards' order files (only the bottom silkscreen changes)
- READMEs: select "Order Number: Specify Position" when ordering; PSU-B
  takes Economic PCBA
Other:
- board text added: "JLCJLCJLCJLC"
Changed lines of the file:
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@@
+		)
+	)
+	(gr_text "JLCJLCJLCJLC"
+		(at 140 160 0)
+		(layer "B.SilkS")
+		(effects
+			(font
+				(size 1 1)
+				(thickness 0.15)
+			)
+			(justify mirror)
 		)
 	)
