File: schematic/hour-meter-psu-b/hour-meter-psu-b.kicad_pcb (KiCad board)
At the start: 2 copper layers, 40 x 30 mm, 24 parts, among them P1 to main J102, U1 TPS54360BDDAR

Commit message: feat(pcb): mark where JLCPCB prints the order number
- New add_order_mark() in the shared board builder: places the
  JLCJLCJLCJLC placeholder (1.0 mm, 0.15 mm stroke) at the free spot
  nearest a given point, clear of pads, holes, courtyards, silkscreen and
  the outline
- Compact board and PSU-B carry it on the bottom silkscreen; their build
  scripts put it back on a rebuild
- Regenerate both boards' order files (only the bottom silkscreen changes)
- READMEs: select "Order Number: Specify Position" when ordering; PSU-B
  takes Economic PCBA
Other:
- board text added: "JLCJLCJLCJLC"
Changed lines of the file:
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@@
+		)
+	)
+	(gr_text "JLCJLCJLCJLC"
+		(at 120 115.5 0)
+		(layer "B.SilkS")
+		(effects
+			(font
+				(size 1 1)
+				(thickness 0.15)
+			)
+			(justify mirror)
 		)
 	)
