File: schematic/hour-meter-board-compact-lm2596/ports.kicad_sch (KiCad schematic)
At the start: 19 parts, among them J801 UART, J802 GPS, J803 QWIIC, J804 EXP, U801 74LVC1G17GW, U802 SRV05-4

Commit message: feat(pcb): use JST VH field connectors on the LM2596 compact board
- J101 (VIN 9-30V), J301 (vehicle IN), J701 (RS485) and J801 (UART) are
  latching JST VH headers instead of screw terminals and JST XH
- add TP101 VIN solder pads in parallel with J101
- GPS J802 becomes a 1x5 male pin header
- re-route the board (U203 VBUS escape fixed by re-routing the USB and
  ESP32 lines under it) and regenerate the JLCPCB order files
- tools-pcb.py: `models` command fetches the JLCPCB/EasyEDA STEP models;
  the downloaded 3d/ folders are git-ignored
Parts:
- J801: footprint Connector_JST:JST_XH_B4B-XH-A_1x04_P2.50mm_Vertical -> Connector_JST:JST_VH_B4P-VH_1x04_P3.96mm_Vertical; LCSC C144395 -> C160317; MPN B4B-XH-A(LF)(SN) -> B4P-VH(LF)(SN)
- J802: footprint Connector_PinSocket_2.54mm:PinSocket_1x05_P2.54mm_Vertical -> Connector_PinHeader_2.54mm:PinHeader_1x05_P2.54mm_Vertical; LCSC C50950 -> C492404; MPN 2.54-1*5PFemale -> PZ254V-11-05P
Changed lines of the file:
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@@
 			)
 		)
-		(property "Footprint" "Connector_JST:JST_XH_B4B-XH-A_1x04_P2.50mm_Vertical"
+		(property "Footprint" "Connector_JST:JST_VH_B4P-VH_1x04_P3.96mm_Vertical"
 			(at 30.48 63.5 0)
 			(hide yes)
@@
 			)
 		)
-		(property "LCSC" "C144395"
+		(property "LCSC" "C160317"
 			(at 30.48 63.5 0)
 			(hide yes)
@@
 			)
 		)
-		(property "MPN" "B4B-XH-A(LF)(SN)"
+		(property "MPN" "B4P-VH(LF)(SN)"
 			(at 30.48 63.5 0)
 			(hide yes)
@@
 			)
 		)
-		(property "Footprint" "Connector_PinSocket_2.54mm:PinSocket_1x05_P2.54mm_Vertical"
+		(property "Footprint" "Connector_PinHeader_2.54mm:PinHeader_1x05_P2.54mm_Vertical"
 			(at 30.48 121.92 0)
 			(hide yes)
@@
 			)
 		)
-		(property "LCSC" "C50950"
+		(property "LCSC" "C492404"
 			(at 30.48 121.92 0)
 			(hide yes)
@@
 			)
 		)
-		(property "MPN" "2.54-1*5PFemale"
+		(property "MPN" "PZ254V-11-05P"
 			(at 30.48 121.92 0)
 			(hide yes)
