File: schematic/hour-meter-board-compact-lm2596/rs485.kicad_sch (KiCad schematic)
At the start: 13 parts, among them J701 RS485, J702 TERM, J703 BIAS, U701 THVD2410DR

Commit message: feat(pcb): use JST VH field connectors on the LM2596 compact board
- J101 (VIN 9-30V), J301 (vehicle IN), J701 (RS485) and J801 (UART) are
  latching JST VH headers instead of screw terminals and JST XH
- add TP101 VIN solder pads in parallel with J101
- GPS J802 becomes a 1x5 male pin header
- re-route the board (U203 VBUS escape fixed by re-routing the USB and
  ESP32 lines under it) and regenerate the JLCPCB order files
- tools-pcb.py: `models` command fetches the JLCPCB/EasyEDA STEP models;
  the downloaded 3d/ folders are git-ignored
Parts:
- J701: footprint TerminalBlock_Phoenix:TerminalBlock_Phoenix_MKDS-1,5-3-5.08_1x03_P5.08mm_Horizontal -> Connector_JST:JST_VH_B3P-VH_1x03_P3.96mm_Vertical; LCSC C474953 -> C160316; MPN KF128-5.08-3P-AA -> B3P-VH(LF)(SN)
Changed lines of the file:
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@@
 			)
 		)
-		(property "Footprint" "TerminalBlock_Phoenix:TerminalBlock_Phoenix_MKDS-1,5-3-5.08_1x03_P5.08mm_Horizontal"
+		(property "Footprint" "Connector_JST:JST_VH_B3P-VH_1x03_P3.96mm_Vertical"
 			(at 256.54 114.3 0)
 			(hide yes)
@@
 			)
 		)
-		(property "LCSC" "C474953"
+		(property "LCSC" "C160316"
 			(at 256.54 114.3 0)
 			(hide yes)
@@
 			)
 		)
-		(property "MPN" "KF128-5.08-3P-AA"
+		(property "MPN" "B3P-VH(LF)(SN)"
 			(at 256.54 114.3 0)
 			(hide yes)
