File: schematic/hour-meter-board-compact-lm2596-io/hour-meter-board-compact-lm2596-io.kicad_pcb (KiCad board)
At the start: 2 copper layers, 80 x 92 mm, 142 parts, among them J101 VIN 9-30V, J201 USB-C, J301 DIN1 DIN2 COM, J501 WP, J701 RS485, J702 TERM, J703 BIAS, J801 UART, J802 GPS, J803 QWIIC, J804 EXP, J902 5V AIN1 GND DOUT1 GND, Q201 MMBT3904, Q202 MMBT3904, SW201 RESET, SW202 BOOT, U101 LM2596S-ADJ, U201 ESP32-WROOM-32E-N4, U202 CH340C, U203 USBLC6-2SC6, U204 AMS1117-3.3, U301 PC817C-S, U302 PC817C-S, U401 DS3231MZ+TRL, U501 AT24C256 DIP-8 (socketed), U601 MPU-6500, U602 LIS3MDLTR, U701 THVD2410DR, U801 74LVC1G17GW, U802 SRV05-4, U901 ADS1115IDGST, U902 SN74AHCT1G125DBVR, U903 BSP75N

Commit message: fix(pcb): link the I/O board's TP101/TP102 solder pads to their nets
- TP101 (VIN) and TP102 (GND) replace the two-hole TP101: 1.5 mm pads on
  the back, above and below J101. They were placed by hand in the PCB
  editor, so they had no symbol link and no net and could not be routed
- they are now library footprints flipped to the bottom and linked to
  their symbols. A 0.5 mm B.Cu track joins J101 pin 1 to TP101, and TP102
  joins the GND pour solid (its thermal spokes were thinner than the
  pour's minimum)
- pours refilled, so the clearance and solder-mask errors are gone:
  DRC 0 errors, 0 unconnected, 0 parity
- tools-pcb.py: TP101/TP102 placed on the bottom side; `reuse` leaves out
  the LM2596 board's route to its two-hole TP101, which would cross TP102
- includes the board move and the KiCad 10 re-save of the sheets
- production: Gerbers and CPL regenerated, BOM unchanged
Parts:
- added TP102: GND, TestPoint:TestPoint_Pad_1.5x1.5mm, B.Cu at (70.5, 114.8)
- TP101: value VIN pads -> VIN; footprint TestPoint:TestPoint_2Pads_Pitch5.08mm_Drill1.3mm -> TestPoint:TestPoint_Pad_1.5x1.5mm; moved to B.Cu
- moved TP101 66.7 mm to (70.5, 101.5), turned to 180 degrees
- moved J902 54.1 mm to (100.6, 143.2)
- moved C601 54.1 mm to (109.8, 63.3)
- moved C604 54.1 mm to (109.8, 67.1)
- moved C901 54.1 mm to (96.5, 145.5)
- moved C902 54.1 mm to (82.7, 146.5)
- moved D901 54.1 mm to (84.0, 141.5)
- moved F803 54.1 mm to (106.0, 117.9)
- moved H103 54.1 mm to (143.0, 105.5)
- moved H105 54.1 mm to (143.4, 145.5)
- moved J101 54.1 mm to (73.5, 106.2)
- moved J803 54.1 mm to (143.4, 113.6)
- moved JP801 54.1 mm to (101.0, 117.9)
- moved R103 54.1 mm to (91.0, 135.5)
- moved R104 54.1 mm to (94.5, 135.5)
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Routing:
- net Net-(J101-Pin_1): track 19.6 -> 13.8 mm

Commit message: feat(pcb): enlarge the I/O board's VIN/GND solder pads to 3 mm
- TP101 (VIN) and TP102 (GND) use TestPoint_Pad_3.0x3.0mm, still on the
  bottom side above and below J101, for hand-soldering 18-22 AWG wire
- keep the GND track from J101 pin 2 to TP102 drawn in pcbnew
- tools-pcb.py: `reuse` leaves out both of the LM2596 board's routes from
  J101 to its two-hole TP101, following only branch-free track chains
- DRC 0 errors / 0 unconnected / 0 parity; Gerbers regenerated, BOM and
  CPL unchanged
Parts:
- TP101, TP102: footprint TestPoint:TestPoint_Pad_1.5x1.5mm -> TestPoint:TestPoint_Pad_3.0x3.0mm
Routing:
- net GND: track 708.4 -> 706.9 mm
Changed lines of the file:
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@@
 		)
 	)
-	(footprint "TestPoint:TestPoint_Pad_1.5x1.5mm"
+	(footprint "TestPoint:TestPoint_Pad_3.0x3.0mm"
 		(layer "B.Cu")
 		(at 70.5 114.75 180)
-		(descr "SMD rectangular pad as test Point, square 1.5mm side length")
+		(descr "SMD rectangular pad as test Point, square 3.0mm side length")
 		(tags "test point SMD pad rectangle square")
 		(property "Reference" "TP102"
-			(at 0 1.648 0)
+			(at 0 2.398 0)
 			(layer "B.SilkS")
 			(hide yes)
@@
 		)
 		(property "Value" "GND"
-			(at 0 -1.75 0)
+			(at 0 -2.55 0)
 			(layer "B.Fab")
 			(effects
@@
 		(duplicate_pad_numbers_are_jumpers no)
 		(fp_line
-			(start 0.95 0.95)
-			(end 0.95 -0.95)
+			(start 1.7 1.7)
+			(end 1.7 -1.7)
 			(stroke
 				(width 0.12)
@@
 		)
 		(fp_line
-			(start 0.95 -0.95)
-			(end -0.95 -0.95)
+			(start 1.7 -1.7)
+			(end -1.7 -1.7)
 			(stroke
 				(width 0.12)
@@
 		)
 		(fp_line
-			(start -0.95 0.95)
-			(end 0.95 0.95)
+			(start -1.7 1.7)
+			(end 1.7 1.7)
 			(stroke
 				(width 0.12)
@@
 		)
 		(fp_line
-			(start -0.95 -0.95)
-			(end -0.95 0.95)
+			(start -1.7 -1.7)
+			(end -1.7 1.7)
 			(stroke
 				(width 0.12)
@@
 		)
 		(fp_line
-			(start 1.25 -1.25)
-			(end 1.25 1.25)
+			(start 2 -2)
+			(end 2 2)
 			(stroke
 				(width 0.05)
@@
 		)
 		(fp_line
-			(start 1.25 -1.25)
-			(end -1.25 -1.25)
+			(start 2 -2)
+			(end -2 -2)
 			(stroke
 				(width 0.05)
@@
 		)
 		(fp_line
-			(start -1.25 1.25)
-			(end 1.25 1.25)
+			(start -2 2)
+			(end 2 2)
 			(stroke
 				(width 0.05)
@@
 		)
 		(fp_line
-			(start -1.25 1.25)
-			(end -1.25 -1.25)
+			(start -2 2)
+			(end -2 -2)
 			(stroke
 				(width 0.05)
@@
 		)
 		(fp_text user "${REFERENCE}"
-			(at 0 1.65 0)
+			(at 0 2.4 0)
 			(layer "B.Fab")
 			(effects
@@
 		(pad "1" smd rect
 			(at 0 0 180)
-			(size 1.5 1.5)
+			(size 3 3)
 			(layers "B.Cu" "B.Mask")
 			(net "GND")
@@
 		(embedded_fonts no)
 	)
-	(footprint "TestPoint:TestPoint_Pad_1.5x1.5mm"
+	(footprint "TestPoint:TestPoint_Pad_3.0x3.0mm"
 		(layer "B.Cu")
 		(at 70.5 101.5 180)
-		(descr "SMD rectangular pad as test Point, square 1.5mm side length")
+		(descr "SMD rectangular pad as test Point, square 3.0mm side length")
 		(tags "test point SMD pad rectangle square")
 		(property "Reference" "TP101"
-			(at 0 1.648 0)
+			(at 0 2.398 0)
 			(layer "B.SilkS")
 			(hide yes)
@@
 		)
 		(property "Value" "VIN"
-			(at 0 -1.75 0)
+			(at 0 -2.55 0)
 			(layer "B.Fab")
 			(effects
@@
 		(duplicate_pad_numbers_are_jumpers no)
 		(fp_line
-			(start 0.95 0.95)
-			(end 0.95 -0.95)
+			(start 1.7 1.7)
+			(end 1.7 -1.7)
 			(stroke
 				(width 0.12)
@@
 		)
 		(fp_line
-			(start 0.95 -0.95)
-			(end -0.95 -0.95)
+			(start 1.7 -1.7)
+			(end -1.7 -1.7)
 			(stroke
 				(width 0.12)
@@
 		)
 		(fp_line
-			(start -0.95 0.95)
-			(end 0.95 0.95)
+			(start -1.7 1.7)
+			(end 1.7 1.7)
 			(stroke
 				(width 0.12)
@@
 		)
 		(fp_line
-			(start -0.95 -0.95)
-			(end -0.95 0.95)
+			(start -1.7 -1.7)
+			(end -1.7 1.7)
 			(stroke
 				(width 0.12)
@@
 		)
 		(fp_line
-			(start 1.25 -1.25)
-			(end 1.25 1.25)
+			(start 2 -2)
+			(end 2 2)
 			(stroke
 				(width 0.05)
@@
 		)
 		(fp_line
-			(start 1.25 -1.25)
-			(end -1.25 -1.25)
+			(start 2 -2)
+			(end -2 -2)
 			(stroke
 				(width 0.05)
@@
 		)
 		(fp_line
-			(start -1.25 1.25)
-			(end 1.25 1.25)
+			(start -2 2)
+			(end 2 2)
 			(stroke
 				(width 0.05)
@@
 		)
 		(fp_line
-			(start -1.25 1.25)
-			(end -1.25 -1.25)
+			(start -2 2)
+			(end -2 -2)
 			(stroke
 				(width 0.05)
@@
 		)
 		(fp_text user "${REFERENCE}"
-			(at 0 1.65 0)
+			(at 0 2.4 0)
 			(layer "B.Fab")
 			(effects
@@
 		(pad "1" smd rect
 			(at 0 0 180)
-			(size 1.5 1.5)
+			(size 3 3)
 			(layers "B.Cu" "B.Mask")
 			(net "Net-(J101-Pin_1)")
@@
 	)
 	(segment
-		(start 114.585 145.42263)
-		(end 116.47 143.53763)
+		(start 73.55 110.12143)
+		(end 70.5 113.17143)
 		(width 0.3)
 		(layer "B.Cu")
@@
 	)
 	(segment
-		(start 91.45 88.79143)
-		(end 93.758 91.09943)
+		(start 114.585 145.42263)
+		(end 116.47 143.53763)
 		(width 0.3)
 		(layer "B.Cu")
@@
 	)
 	(segment
-		(start 75.59 112.16143)
-		(end 73.55 110.12143)
+		(start 91.45 88.79143)
+		(end 93.758 91.09943)
 		(width 0.3)
 		(layer "B.Cu")
@@
 	)
 	(segment
-		(start 75.59 116.64143)
-		(end 75.59 112.16143)
+		(start 77.85 105.82143)
+		(end 77.85 100.40143)
 		(width 0.3)
 		(layer "B.Cu")
@@
 	)
 	(segment
-		(start 77.85 105.82143)
-		(end 77.85 100.40143)
+		(start 70.5 113.17143)
+		(end 70.5 114.75)
 		(width 0.3)
 		(layer "B.Cu")
