File: schematic/hour-meter-board-microfit/eeprom-at24c256.kicad_sch (KiCad schematic)
At the start: 4 parts, among them J501 WP, U501 AT24C256 DIP-8 (socketed)

Commit message: feat(pcb): wire the Micro-Fit board's field I/O through one J1 harness
- New Harness sheet: J1 Molex Micro-Fit 3.0 2x7 right-angle header
  (43045-1400, LCSC C277677) replaces J101, J301, J701, J801 and J902.
- Pin order: VIN, AIN1, DOUT1, DIN1 and DIN2 sit on the back row (8-14)
  so their 0.8 mm Vehicle clearance never has to fit between two pads.
  The isolated DIN group (DIN1, DIN2 and two DIN COM pins 6/7) fills
  the pin 7/14 end, next to RS485 A/B, which are rated +/-70 V.
- J802 GPS becomes a JST GH 6-pin in the Pixhawk pinout with I2C;
  PPS moves to the TP801 solder pad.
- The J804 expansion header becomes test pads TP802-TP808; F802 and
  F902 go. J501, J702 and J703 become solder jumpers JP501, JP702-JP704.
- U501 is now the SOIC-8 AT24C256C-SSHL-T (C6482); TP101/TP102 dropped.
- Net-class patterns follow the renamed root nets; ERC shows only the
  two known IMU warnings.
Parts:
- removed J501: WP, Connector_PinHeader_2.54mm:PinHeader_1x02_P2.54mm_Vertical, symbol Connector_Generic:Conn_01x02
- added JP501: WP, Jumper:SolderJumper-2_P1.3mm_Open_RoundedPad1.0x1.5mm, symbol Jumper:SolderJumper_2_Open
- U501: value AT24C256 DIP-8 (socketed) -> AT24C256C-SSHL-T; footprint Package_DIP:DIP-8_W7.62mm_Socket -> Package_SO:SOIC-8_3.9x4.9mm_P1.27mm; Fitted AT24C256 DIP-8 inserted by the user (e.g. LCSC C434602 AT24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 -> Assembled by JLCPCB (SOIC-8, LCSC C6482); LCSC C2874007 -> C6482; MPN IC254V-12-08-0743 -> AT24C256C-SSHL-T
Connections:
- net +3V3: now also JP501.2 (B)
- net EE_WP: now also JP501.1 (A)
Other:
- note added: "EEPROM (replaces AT24C256 module) U501 AT24C256C-SSHL-T (SOIC-8, LCSC C6482) is assembled by JLCPCB. I2C address 0x50 (A0 = A1 = A2 = GND). The firmware layout is fixed at 32 KB (EepromLayout.h), so fit a 24C256 or 24C512. WP: R501 10k pulls EE_WP low (writes enabled); bridging solder jumper JP501 ties WP to +3V3 and write-protects the chip. No I2C pull-ups here (they are on esp32-core)."
- note removed: "EEPROM (replaces AT24C256 module) U501 is a swappable chip in a DIP-8 socket (only the socket is assembled): the user inserts an AT24C256 DIP-8, e.g. LCSC C434602 AT24C256N or C411624 24LC256-I/P. I2C address 0x50 (A0 = A1 = A2 = GND). The firmware layout is fixed at 32 KB (EepromLayout.h), so fit a 24C256 or 24C512. WP: R501 10k pulls EE_WP low (writes enabled); a jumper on J501 ties WP to +3V3 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"
