File: schematic/hour-meter-board-microfit/io.kicad_sch (KiCad schematic)
At the start: 15 parts, among them J902 5V AIN1 GND DOUT1 GND, U901 ADS1115IDGST, U902 SN74AHCT1G125DBVR, U903 BSP75N

Commit message: feat(pcb): wire the Micro-Fit board's field I/O through one J1 harness
- New Harness sheet: J1 Molex Micro-Fit 3.0 2x7 right-angle header
  (43045-1400, LCSC C277677) replaces J101, J301, J701, J801 and J902.
- Pin order: VIN, AIN1, DOUT1, DIN1 and DIN2 sit on the back row (8-14)
  so their 0.8 mm Vehicle clearance never has to fit between two pads.
  The isolated DIN group (DIN1, DIN2 and two DIN COM pins 6/7) fills
  the pin 7/14 end, next to RS485 A/B, which are rated +/-70 V.
- J802 GPS becomes a JST GH 6-pin in the Pixhawk pinout with I2C;
  PPS moves to the TP801 solder pad.
- The J804 expansion header becomes test pads TP802-TP808; F802 and
  F902 go. J501, J702 and J703 become solder jumpers JP501, JP702-JP704.
- U501 is now the SOIC-8 AT24C256C-SSHL-T (C6482); TP101/TP102 dropped.
- Net-class patterns follow the renamed root nets; ERC shows only the
  two known IMU warnings.
Parts:
- removed F902: 0.2A, Fuse:Fuse_1206_3216Metric, symbol Device:Polyfuse
- removed J902: 5V AIN1 GND DOUT1 GND, Connector_JST:JST_VH_B5P-VH_1x05_P3.96mm_Vertical, symbol Connector:Screw_Terminal_01x05
Other:
- note added: "I/O on J1 (Harness sheet): AIN1 = J1 pin 9 (sensor return: J1 pin 2), DOUT1 = J1 pin 10; sensor 5 V from J1 pin 11 (200 mA via F801). NOT isolated: GND is the supply ground (vehicle battery negative). AIN1: 0-30 V measured (abs. max +/-60 V continuous), input resistance 110 kOhm. 2 x 49.9k 0.1 % 1206 in series (shares a 600 V pulse) / 10k 0.1 %: ratio 0.0911, 30 V -> 2.73 V. ADS1115 (I2C 0x48, AI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"
- note removed: "I/O PORT J902 (JST VH 5-pin): 1 +5V_OUT (200 mA PTC), 2 AIN1, 3 GND, 4 DOUT1, 5 GND. NOT isolated: GND is the supply ground (J101-2, vehicle battery negative). AIN1: 0-30 V measured (abs. max +/-60 V continuous), input resistance 110 kOhm. 2 x 49.9k 0.1 % 1206 in series (shares a 600 V pulse) / 10k 0.1 %: ratio 0.0911, 30 V -> 2.73 V. ADS1115 (I2C 0x48, AIN0) PGA ranges: +/-4.096 V -> 0-36 V (VDD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"
