File: schematic/hour-meter-board-microfit/opto-inputs.kicad_sch (KiCad schematic)
At the start: 19 parts, among them J301 DIN1 DIN2 COM, U301 PC817C-S, U302 PC817C-S

Commit message: feat(pcb): wire the Micro-Fit board's field I/O through one J1 harness
- New Harness sheet: J1 Molex Micro-Fit 3.0 2x7 right-angle header
  (43045-1400, LCSC C277677) replaces J101, J301, J701, J801 and J902.
- Pin order: VIN, AIN1, DOUT1, DIN1 and DIN2 sit on the back row (8-14)
  so their 0.8 mm Vehicle clearance never has to fit between two pads.
  The isolated DIN group (DIN1, DIN2 and two DIN COM pins 6/7) fills
  the pin 7/14 end, next to RS485 A/B, which are rated +/-70 V.
- J802 GPS becomes a JST GH 6-pin in the Pixhawk pinout with I2C;
  PPS moves to the TP801 solder pad.
- The J804 expansion header becomes test pads TP802-TP808; F802 and
  F902 go. J501, J702 and J703 become solder jumpers JP501, JP702-JP704.
- U501 is now the SOIC-8 AT24C256C-SSHL-T (C6482); TP101/TP102 dropped.
- Net-class patterns follow the renamed root nets; ERC shows only the
  two known IMU warnings.
Parts:
- removed J301: DIN1 DIN2 COM, Connector_JST:JST_VH_B3P-VH_1x03_P3.96mm_Vertical, symbol Connector:Screw_Terminal_01x03
