File: schematic/hour-meter-board-microfit/power-input.kicad_sch (KiCad schematic)
At the start: 26 parts, among them J101 VIN 9-30V, U101 LM2596S-ADJ

Commit message: feat(pcb): wire the Micro-Fit board's field I/O through one J1 harness
- New Harness sheet: J1 Molex Micro-Fit 3.0 2x7 right-angle header
  (43045-1400, LCSC C277677) replaces J101, J301, J701, J801 and J902.
- Pin order: VIN, AIN1, DOUT1, DIN1 and DIN2 sit on the back row (8-14)
  so their 0.8 mm Vehicle clearance never has to fit between two pads.
  The isolated DIN group (DIN1, DIN2 and two DIN COM pins 6/7) fills
  the pin 7/14 end, next to RS485 A/B, which are rated +/-70 V.
- J802 GPS becomes a JST GH 6-pin in the Pixhawk pinout with I2C;
  PPS moves to the TP801 solder pad.
- The J804 expansion header becomes test pads TP802-TP808; F802 and
  F902 go. J501, J702 and J703 become solder jumpers JP501, JP702-JP704.
- U501 is now the SOIC-8 AT24C256C-SSHL-T (C6482); TP101/TP102 dropped.
- Net-class patterns follow the renamed root nets; ERC shows only the
  two known IMU warnings.
Parts:
- removed J101: VIN 9-30V, Connector_JST:JST_VH_B2P-VH_1x02_P3.96mm_Vertical, symbol Connector:Screw_Terminal_01x02
- removed TP101: VIN, TestPoint:TestPoint_Pad_3.0x3.0mm, symbol Connector:TestPoint
- removed TP102: GND, TestPoint:TestPoint_Pad_3.0x3.0mm, symbol Connector:TestPoint
Connections:
- net VIN_IN: now reaches F101.1
Other:
- note added: "POWER INPUT Vehicle supply 9-30 V on J1 pin 8 (VIN_IN, Harness sheet); the return is the J1 GND pins 1 and 2. F101 PTC -> D103 reverse block -> D104 TVS (SMAJ30CA) -> U101 LM2596S-ADJ, 5.29 V on +5V_PSU (R103/R104 = 3.3k/1k). +5V_PSU -> D101 SS34 -> +5V. USB VBUS is OR-ed into +5V on the esp32-core sheet. VIN_SENSE = VIN x 5.6/105.6 (GPIO34, ADC1_CH6). H102-H105 = board corner holes."
- note removed: "POWER INPUT Vehicle supply 9-30 V on J101 (JST VH) or on the TP101 solder pads: same net, use one of them. F101 PTC -> D103 reverse block -> D104 TVS (SMAJ30CA) -> U101 LM2596S-ADJ, 5.29 V on +5V_PSU (R103/R104 = 3.3k/1k). +5V_PSU -> D101 SS34 -> +5V. USB VBUS is OR-ed into +5V on the esp32-core sheet. VIN_SENSE = VIN x 5.6/105.6 (GPIO34, ADC1_CH6). H102-H105 = board corner holes."
