File: schematic/hour-meter-board-microfit/rs485.kicad_sch (KiCad schematic)
At the start: 13 parts, among them J701 RS485, J702 TERM, J703 BIAS, U701 THVD2410DR

Commit message: feat(pcb): wire the Micro-Fit board's field I/O through one J1 harness
- New Harness sheet: J1 Molex Micro-Fit 3.0 2x7 right-angle header
  (43045-1400, LCSC C277677) replaces J101, J301, J701, J801 and J902.
- Pin order: VIN, AIN1, DOUT1, DIN1 and DIN2 sit on the back row (8-14)
  so their 0.8 mm Vehicle clearance never has to fit between two pads.
  The isolated DIN group (DIN1, DIN2 and two DIN COM pins 6/7) fills
  the pin 7/14 end, next to RS485 A/B, which are rated +/-70 V.
- J802 GPS becomes a JST GH 6-pin in the Pixhawk pinout with I2C;
  PPS moves to the TP801 solder pad.
- The J804 expansion header becomes test pads TP802-TP808; F802 and
  F902 go. J501, J702 and J703 become solder jumpers JP501, JP702-JP704.
- U501 is now the SOIC-8 AT24C256C-SSHL-T (C6482); TP101/TP102 dropped.
- Net-class patterns follow the renamed root nets; ERC shows only the
  two known IMU warnings.
Parts:
- removed J701: RS485, Connector_JST:JST_VH_B3P-VH_1x03_P3.96mm_Vertical, symbol Connector:Screw_Terminal_01x03
- removed J702: TERM, Connector_PinHeader_2.54mm:PinHeader_1x02_P2.54mm_Vertical, symbol Connector_Generic:Conn_01x02
- removed J703: BIAS, Connector_PinHeader_2.54mm:PinHeader_2x02_P2.54mm_Vertical, symbol Connector_Generic:Conn_02x02_Odd_Even
- added JP702: TERM 120R, Jumper:SolderJumper-2_P1.3mm_Open_RoundedPad1.0x1.5mm, symbol Jumper:SolderJumper_2_Open
- added JP703: BIAS A, Jumper:SolderJumper-2_P1.3mm_Open_RoundedPad1.0x1.5mm, symbol Jumper:SolderJumper_2_Open
- added JP704: BIAS B, Jumper:SolderJumper-2_P1.3mm_Open_RoundedPad1.0x1.5mm, symbol Jumper:SolderJumper_2_Open
Connections:
- net +3V3: now also JP703.1 (A)
- net BIAS_A: now also JP703.2 (B)
- net BIAS_B: now also JP704.1 (A)
- net GND: now also JP704.2 (B)
- net RS485_B: now also JP702.2 (B)
- net TERM_A: now also JP702.1 (A)
Other:
- note added: "RS485 (replaces MAX485 module), fault-protected U701 THVD2410DR 3.3 V half-duplex transceiver on UART1: GPIO4 = TX (D), GPIO35 = RX (R), GPIO25 = DE + /RE (ESP-IDF UART RS485 half-duplex mode). A and B are rated +/-70 V and work over +/-25 V common mode, so a bus wire shorted to the 12 V or 24 V supply does no damage. A = J1 pin 5, B = J1 pin 12 (Harness sheet). R701 / R702 hold RX / TX high (R f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"
- note removed: "RS485 (replaces MAX485 module), fault-protected U701 THVD2410DR 3.3 V half-duplex transceiver on UART1: GPIO4 = TX (D), GPIO35 = RX (R), GPIO25 = DE + /RE (ESP-IDF UART RS485 half-duplex mode). A and B are rated +/-70 V and work over +/-25 V common mode, so a bus wire shorted to the 12 V or 24 V supply does no damage. R701 / R702 hold RX / TX high (R floats while transmitting); R703 holds DE low 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"
