File: schematic/hour-meter-board-microfit/ports.kicad_sch (KiCad schematic)
At the start: 19 parts, among them J801 UART, J802 GPS, J803 QWIIC, J804 EXP, U801 74LVC1G17GW, U802 SRV05-4

Commit message: feat(pcb): wire the Micro-Fit board's field I/O through one J1 harness
- New Harness sheet: J1 Molex Micro-Fit 3.0 2x7 right-angle header
  (43045-1400, LCSC C277677) replaces J101, J301, J701, J801 and J902.
- Pin order: VIN, AIN1, DOUT1, DIN1 and DIN2 sit on the back row (8-14)
  so their 0.8 mm Vehicle clearance never has to fit between two pads.
  The isolated DIN group (DIN1, DIN2 and two DIN COM pins 6/7) fills
  the pin 7/14 end, next to RS485 A/B, which are rated +/-70 V.
- J802 GPS becomes a JST GH 6-pin in the Pixhawk pinout with I2C;
  PPS moves to the TP801 solder pad.
- The J804 expansion header becomes test pads TP802-TP808; F802 and
  F902 go. J501, J702 and J703 become solder jumpers JP501, JP702-JP704.
- U501 is now the SOIC-8 AT24C256C-SSHL-T (C6482); TP101/TP102 dropped.
- Net-class patterns follow the renamed root nets; ERC shows only the
  two known IMU warnings.
Parts:
- removed F802: 0.2A, Fuse:Fuse_1206_3216Metric, symbol Device:Polyfuse
- removed J801: UART, Connector_JST:JST_VH_B4P-VH_1x04_P3.96mm_Vertical, symbol Connector_Generic:Conn_01x04
- removed J804: EXP, Connector_PinHeader_2.54mm:PinHeader_2x05_P2.54mm_Vertical, symbol Connector_Generic:Conn_02x05_Odd_Even
- added TP801: PPS, TestPoint:TestPoint_Pad_D1.0mm, symbol Connector:TestPoint
- added TP802: IO5, TestPoint:TestPoint_Pad_D1.0mm, symbol Connector:TestPoint
- added TP803: IO15, TestPoint:TestPoint_Pad_D1.0mm, symbol Connector:TestPoint
- added TP804: IO18, TestPoint:TestPoint_Pad_D1.0mm, symbol Connector:TestPoint
- added TP805: IO19, TestPoint:TestPoint_Pad_D1.0mm, symbol Connector:TestPoint
- added TP806: IO33, TestPoint:TestPoint_Pad_D1.0mm, symbol Connector:TestPoint
- added TP807: +3V3, TestPoint:TestPoint_Pad_D1.0mm, symbol Connector:TestPoint
- added TP808: GND, TestPoint:TestPoint_Pad_D1.0mm, symbol Connector:TestPoint
- J802: value GPS -> GPS (GH 6-pin); footprint Connector_PinHeader_2.54mm:PinHeader_1x05_P2.54mm_Vertical -> Connector_JST:JST_GH_SM06B-GHS-TB_1x06-1MP_P1.25mm_Horizontal; symbol Connector_Generic:Conn_01x05 -> Connector_Generic_MountingPin:Conn_01x06_MountingPin; LCSC C492404 -> C133065; MPN PZ254V-11-05P -> SM06B-GHS-TB(LF)(SN)
Connections:
- net +3V3: now also TP807.1
- net EXP_IO15: now also TP803.1
- net EXP_IO18: now also TP804.1
- net EXP_IO19: now also TP805.1
- net EXP_IO33: now also TP806.1
- net EXP_IO5: now also TP802.1
- net GND: now also J802.6 (Pin_6), J802.MP (MountPin), TP808.1; no longer J802.2 (Pin_2)
- net GPS_PPS_EXT: now also TP801.1; no longer J802.5 (Pin_5)
- net GPS_RX_EXT: now also J802.2 (Pin_2); no longer J802.4 (Pin_4)
- net I2C_SCL: now also J802.4 (Pin_4)
- net I2C_SDA: now also J802.5 (Pin_5)
- no-connect marks 1 -> 0
Other:
- note added: "J802 GPS port: JST GH 6-pin, Pixhawk GPS pinout: 1 VCC, 2 TX (to GPS RX), 3 RX (from GPS TX), 4 SCL, 5 SDA, 6 GND. 100R series on the UART (GPIO36 / GPIO32); SCL/SDA (GPS compass) share the board I2C bus. PPS (GPIO39) is the TP801 solder pad. R806 holds GPS_TXD high with no module (GPIO36 has no pull-up); R807 holds PPS low. GPS supply = 3V3 by default (JP801 1-2); cut 1-2 and bridge 2-3 for a 5 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"
- note added: "PORTS UART sensor port on J1 (Harness sheet): pin 3 TX, pin 4 RX, pin 2 GND, pin 11 = 5 V, 200 mA via F801 polyfuse (shared with AIN1 sensors). UART2 = GPIO17 TX (3.3 V out via R801 100R) / GPIO16 RX via U801 74LVC1G17 (5 V-tolerant input, R802 keeps it idle-high). U802 SRV05-4 = ESD on the four external UART/GPS lines. The port data lines are 3.3/5 V logic: they survive ESD, not a wire to the ve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"
- note removed: "PORTS J801 UART sensor port: UART2 = GPIO17 TX (3.3 V out via R801 100R) / GPIO16 RX via U801 74LVC1G17 (5 V-tolerant input, R802 keeps it idle-high); pin 1 = 5 V, 200 mA via F801 polyfuse. U802 SRV05-4 = ESD on the four external UART/GPS lines. J802 GPS card header for u-blox type modules: UART on GPIO36 (GPS TX) / GPIO32 (GPS RX), PPS on GPIO39, 100R series. R806 holds GPS_TXD high with no modu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"

Commit message: feat(pcb): add three side-view indicator LEDs to the Micro-Fit board
- D801 P1 (green, GPIO18) and D802 P2 (yellow, GPIO19) are process
  indicators; D803 USER (blue, GPIO5) is free for the program. They are
  Lite-On LTST-S270 side-view LEDs on the right edge below H103, lenses
  at the board edge, 330R each, active high. GPIO5/18/19 were the test
  pads TP802/TP804/TP805.
- tools-pcb.py: `update` adds and removes parts on the routed board;
  `route`, `finish`, `update` and `silk` follow a board moved in KiCad
  (offset measured on U601); add_pinout draws the two-column J1 pinout.
- Keeps the KiCad edits made after the layout commit: the board moved
  by (18.20, -48.27) mm and the bottom-silkscreen pinout split into two
  columns.
- DRC 0 errors, 0 unconnected, 0 parity; BOM 71 lines, CPL 131, all in
  stock for 10 boards.
Parts:
- removed TP802: IO5, TestPoint:TestPoint_Pad_D1.0mm, symbol Connector:TestPoint
- removed TP804: IO18, TestPoint:TestPoint_Pad_D1.0mm, symbol Connector:TestPoint
- removed TP805: IO19, TestPoint:TestPoint_Pad_D1.0mm, symbol Connector:TestPoint
- added D801: P1 (green), LED_SMD:LED_Kingbright_APA1606_1.6x0.6mm_Horizontal, symbol Device:LED
- added D802: P2 (yellow), LED_SMD:LED_Kingbright_APA1606_1.6x0.6mm_Horizontal, symbol Device:LED
- added D803: USER (blue), LED_SMD:LED_Kingbright_APA1606_1.6x0.6mm_Horizontal, symbol Device:LED
- added R808, R809, R810: 330R, Resistor_SMD:R_0603_1608Metric, symbol Device:R
Connections:
- net EXP_IO18: now also R808.1
- net EXP_IO19: now also R809.1
- net EXP_IO5: now also R810.1
- net GND: now also D801.1 (K), D802.1 (K), D803.1 (K)
- new net: D803.2 (A), R810.2
- new net: D802.2 (A), R809.2
- new net: D801.2 (A), R808.2
Other:
- note added: "INDICATOR LEDS: side-view Lite-On LTST-S270 (1.6 x 1.2 mm) on the right board edge, lighting out through the case wall. Active high: GPIO = 1 -> LED on, 2-4 mA through 330R. D801 P1 green (GPIO18), D802 P2 yellow (GPIO19): process. D803 USER blue (GPIO5): free for the program. GPIO5 is a strapping pin (SDIO slave timing only, unused); it may flicker at boot."

Commit message: feat(pcb): one green LED part and a pinout spec for the Micro-Fit board
D802 and D803 become the green LTST-S270TGKT, like D801. Its JLCPCB
model faces the board edge like the KiCad footprint, where the yellow
and blue parts' models faced the other way, and one LED part means two
fewer extended parts. `update` now also brings the value and fields of
parts that stay in line with the schematic.

PINOUT.md gives every J1 pin's working range, absolute maximum and
current, the other ports, the I2C addresses in use, and the power
budget at 12 V: 0.5 W idle, 0.8 W typical, about 4 W with every port
at its limit. The trucks feed the board from a 24 -> 12 V converter.
Parts:
- D802: value P2 (yellow) -> P2 (green); LCSC C133119 -> C364567; MPN LTST-S270KSKT -> LTST-S270TGKT
- D803: value USER (blue) -> USER (green); LCSC C125115 -> C364567; MPN LTST-S270TBKT -> LTST-S270TGKT
Other:
- note added: "INDICATOR LEDS: side-view Lite-On LTST-S270TGKT, green (1.6 x 1.2 mm), on the right board edge, lighting out through the case wall. One colour: its JLCPCB footprint and model face the edge like the KiCad footprint. Active high: GPIO = 1 -> LED on, about 1.7 mA through 330R. D801 P1 (GPIO18), D802 P2 (GPIO19): process. D803 USER (GPIO5): free for the program. GPIO5 is a strapping pin (SDIO slave t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"
- note removed: "INDICATOR LEDS: side-view Lite-On LTST-S270 (1.6 x 1.2 mm) on the right board edge, lighting out through the case wall. Active high: GPIO = 1 -> LED on, 2-4 mA through 330R. D801 P1 green (GPIO18), D802 P2 yellow (GPIO19): process. D803 USER blue (GPIO5): free for the program. GPIO5 is a strapping pin (SDIO slave timing only, unused); it may flicker at boot."
Changed lines of the file:
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@@
     (effects (font (size 1.5 1.5)) (justify left top))
   )
-  (text "INDICATOR LEDS: side-view Lite-On LTST-S270 (1.6 x 1.2 mm) on the\nright board edge, lighting out through the case wall.\nActive high: GPIO = 1 -> LED on, 2-4 mA through 330R.\nD801 P1 green (GPIO18), D802 P2 yellow (GPIO19): process.\nD803 USER blue (GPIO5): free for the program. GPIO5 is a strapping\npin (SDIO slave timing only, unused); it may flicker at boot."
+  (text "INDICATOR LEDS: side-view Lite-On LTST-S270TGKT, green (1.6 x 1.2 mm),\non the right board edge, lighting out through the case wall. One colour:\nits JLCPCB footprint and model face the edge like the KiCad footprint.\nActive high: GPIO = 1 -> LED on, about 1.7 mA through 330R.\nD801 P1 (GPIO18), D802 P2 (GPIO19): process.\nD803 USER (GPIO5): free for the program. GPIO5 is a strapping\npin (SDIO slave timing only, unused); it may flicker at boot."
     (at 25.4 177.8 0)
     (effects (font (size 1.5 1.5)) (justify left top))
@@
 			)
 		)
-		(property "Value" "P2 (yellow)"
+		(property "Value" "P2 (green)"
 			(at 167.64 184.15 0)
 			(effects
@@
 			)
 		)
-		(property "Description" "Side-view LED, yellow, 1.6 x 1.2 mm (Lite-On LTST-S270); lights out of the right board edge"
+		(property "Description" "Side-view LED, green, 1.6 x 1.2 mm (Lite-On LTST-S270); lights out of the right board edge"
 			(at 146.05 184.15 0)
 			(hide yes)
@@
 			)
 		)
-		(property "LCSC" "C133119"
+		(property "LCSC" "C364567"
 			(at 146.05 184.15 0)
 			(hide yes)
@@
 			)
 		)
-		(property "MPN" "LTST-S270KSKT"
+		(property "MPN" "LTST-S270TGKT"
 			(at 146.05 184.15 0)
 			(hide yes)
@@
 			)
 		)
-		(property "Value" "USER (blue)"
+		(property "Value" "USER (green)"
 			(at 167.64 190.5 0)
 			(effects
@@
 			)
 		)
-		(property "Description" "Side-view LED, blue, 1.6 x 1.2 mm (Lite-On LTST-S270); lights out of the right board edge"
+		(property "Description" "Side-view LED, green, 1.6 x 1.2 mm (Lite-On LTST-S270); lights out of the right board edge"
 			(at 146.05 190.5 0)
 			(hide yes)
@@
 			)
 		)
-		(property "LCSC" "C125115"
+		(property "LCSC" "C364567"
 			(at 146.05 190.5 0)
 			(hide yes)
@@
 			)
 		)
-		(property "MPN" "LTST-S270TBKT"
+		(property "MPN" "LTST-S270TGKT"
 			(at 146.05 190.5 0)
 			(hide yes)
